File: hardware/hackxpansion/pcb/module.kicad_sch (KiCad schematic)
At the start: 4 parts

Commit message: started moving resistors from daughter to main board
Parts:
- removed R11, R16: 10k, Resistor_SMD:R_0402_1005Metric, symbol Device:R
- removed R26: 5R1, Resistor_SMD:R_0402_1005Metric, symbol Device:R
Connections:
- net +3V3: now also U1.2 (3V3)
