File: hardware/hackxpansion/pcb/hackxpansion.kicad_pcb (KiCad board)
At the start: 4 copper layers, 52 x 69 mm, 103 parts, among them CN1 533981471, CN2 533981471, CN3 533981471, CN4 533981471, IC1 ADS7128IRTET, J2 USB_C_Receptacle_USB2.0_14P, J3 Conn_ARM_JTAG_SWD_10, Q1 BSS138, Q2 2N7002, SW1 SW_Push, SW2 SW_Push, SW3 SW_On_Off, U2 RP2354B, U5 SPX3819M5-L-3-3, U7 BQ24075RGT, U8 USBLC6-2SC6, Y1 ABM8-272-T3

Commit message: started moving resistors from daughter to main board
Parts:
- removed R16, R17: 10k, Resistor_SMD:R_0402_1005Metric
- removed R26, R27, R28, R29: 5R1, Resistor_SMD:R_0402_1005Metric
- added R30: 10k, Resistor_SMD:R_0402_1005Metric, F.Cu at (93.4, 71.8)
- added R31: 10k, Resistor_SMD:R_0402_1005Metric, F.Cu at (93.4, 73.8)
- added R32: 10k, Resistor_SMD:R_0402_1005Metric, F.Cu at (93.4, 75.7)
- added R33: 10k, Resistor_SMD:R_0402_1005Metric, F.Cu at (93.4, 77.7)
- added R36: 5R1, Resistor_SMD:R_0402_1005Metric, F.Cu at (122.4, 94.7)
- added R37: 5R1, Resistor_SMD:R_0402_1005Metric, F.Cu at (148.7, 94.1)
- R11, R12: value 10k -> 5R1
- moved R18 38.9 mm to (109.7, 67.1), turned to 180 degrees
- moved R20 32.8 mm to (109.7, 66.2)
- moved R19 30.7 mm to (109.7, 69.3), turned to 180 degrees
- moved R21 23.5 mm to (109.9, 68.4)
- moved R11 23.3 mm to (132.6, 64.6), turned to 0 degrees
- moved R12 3.15 mm to (107.2, 64.2), turned to 90 degrees
Connections:
- CN1 pad 13: /DAUGHT_+3V3 -> /Daughter Board/+3V3_MOD2
- CN2 pad 13: /+3V3 -> /Connector Main Mod3/+3V3
- CN3 pad 13: /+3V3 -> /Connector Main Mod2/+3V3
- CN4 pad 13: /DAUGHT_+3V3 -> /Daughter Board/+3V3_MOD3
- R11 pad 1: /Main Board/ADC/mod0.MD0 -> /+3V3
- R11 pad 2: /GND -> /Connector Main Mod2/+3V3
- R12 pad 1: /Main Board/ADC/mod1.MD0 -> /+3V3
- R12 pad 2: /GND -> /Connector Main Mod3/+3V3
- R18 pad 1: /Connector Daughter Mod2/mod.MD1 -> /Main Board/ADC/mod1.MD1
- R18 pad 2: /DAUGHT_GND -> /GND
- R19 pad 1: /Connector Daughter Mod3/mod.MD1 -> /Main Board/ADC/mod0.MD1
- R19 pad 2: /DAUGHT_GND -> /GND
- R20 pad 1: /Connector Daughter Mod2/mod.MD0 -> /Main Board/ADC/mod1.MD0
- R20 pad 2: /DAUGHT_GND -> /GND
- R21 pad 1: /Connector Daughter Mod3/mod.MD0 -> /Main Board/ADC/mod0.MD0
- R21 pad 2: /DAUGHT_GND -> /GND
- U1 pad 2: Net-(U1-3V3) -> /Main Board/Module Bay 0/+3V3
- U3 pad 2: Net-(U3-3V3) -> /Main Board/Module Bay 1/+3V3
- U4 pad 2: Net-(U4-3V3) -> /Daughter Board/+3V3_MOD2
- U6 pad 2: Net-(U6-3V3) -> /Daughter Board/+3V3_MOD3
Routing:
- net /+3V3: track 297.4 -> 363.6 mm, vias 16 -> 21
- net /DAUGHT_+3V3: track 63.4 -> 0.00 mm, vias 4 -> 0
- net /Connector Main Mod2/+3V3: track 0.00 -> 2.92 mm
- net Net-(U3-3V3): track 2.67 -> 0.00 mm
- net Net-(U4-3V3): track 2.64 -> 0.00 mm
- net /Daughter Board/+3V3_MOD2: track 0.00 -> 2.64 mm
- net Net-(U6-3V3): track 2.50 -> 0.00 mm
- net /Daughter Board/+3V3_MOD3: track 0.00 -> 2.50 mm
- net /GND: track 65.8 -> 63.5 mm, vias 417 -> 419
- net /Main Board/Module Bay 1/+3V3: track 0.00 -> 2.30 mm
- net Net-(U1-3V3): track 2.13 -> 0.00 mm
- net /Main Board/Module Bay 0/+3V3: track 0.00 -> 2.13 mm
- net /DAUGHT_GND: track 8.75 -> 7.51 mm, vias 187 -> 185
- net /Connector Main Mod3/+3V3: track 0.00 -> 1.07 mm
- net /Main Board/ADC/mod1.MD0: track 79.0 -> 79.6 mm

Commit message: placed resisotrs on main board
Parts:
- moved R31 31.6 mm to (123.7, 64.8), turned to -45 degrees
- moved R30 27.8 mm to (120.3, 64.7), turned to -90 degrees
- moved R33 21.2 mm to (109.7, 64.2), turned to 180 degrees
- moved R32 17.9 mm to (110.9, 72.1), turned to -90 degrees
Routing:
- net /+3V3: track 363.6 -> 300.2 mm, vias 21 -> 17
- net /Daughter Board/+3V3_MOD2: track 2.64 -> 28.4 mm, vias 0 -> 1
- net /Daughter Board/+3V3_MOD3: track 2.50 -> 25.7 mm, vias 0 -> 1
- net /DAUGHT_GND: track 7.51 -> 1.12 mm, vias 185 -> 203
- net /Connector Daughter Mod2/mod.MD0: track 20.5 -> 18.0 mm
- net /Connector Daughter Mod3/mod.MD0: track 15.8 -> 13.5 mm
- net /Connector Daughter Mod2/mod.MD1: track 21.6 -> 20.0 mm
- net /Connector Daughter Mod3/mod.MD1: track 19.0 -> 17.4 mm
- net /Connector Main Mod2/mod.MD1: track 35.3 -> 36.3 mm, vias 2 -> 3
- net /Connector Main Mod2/mod.MD0: track 35.3 -> 36.2 mm, vias 2 -> 3
- net /GND: track 63.5 -> 63.1 mm, vias 419 -> 416
