File: hardware/hackxpansion/pcb/pwr.kicad_sch (KiCad schematic)
At the start: 18 parts, among them Q2 2N7002, SW3 SW_On_Off, U5 SPX3819M5-L-3-3, U7 BQ24075RGT

Commit message: added more vias, and repaced 100k with 10k
Parts:
- R15: value 100k -> 10k; LCSC C481918 -> C190095
Changed lines of the file:
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@@
 			)
 		)
-		(property "Value" "100k"
+		(property "Value" "10k"
 			(at 31.75 102.8699 0)
 			(show_name no)
@@
 			)
 		)
-		(property "LCSC" "C481918"
+		(property "LCSC" "C190095"
 			(at 34.29 101.6 0)
 			(hide yes)
